File: KiCad/Headers.sch (KiCad schematic (older format))
At the start: 5 parts, among them CON1 AVR-JTAG-10, J23 Debug Log, J24 ISP0, J25 ISP1, J26 NeoPixel

Commit message: More work
Parts:
- removed J23: Debug Log, symbol CONN_01X01
- removed J26: NeoPixel, symbol CONN_01X01
- added J603, J604, J607, J608: CONN_01X02, Pin_Headers:Pin_Header_Straight_1x02_Pitch2.54mm, symbol CONN_01X02
- added J609, J610: CONN_01X03, Pin_Headers:Pin_Header_Straight_1x03_Pitch2.54mm, symbol CONN_01X03
- renumbered CON1 to CON601, J24 to J601, J25 to J602
Connections:
- net GND: now also J603.1 (P1), J604.1 (P1), J607.1 (P1), J608.1 (P1), J609.1 (P1), J610.1 (P1)
- new net GPI38: J603.2 (P2)
- new net GPI39: J604.2 (P2)
- new net GPIO/1UART0_TX: J609.2 (P2)
- new net GPIO0/Button: J608.2 (P2)
- new net GPIO16/UART2_RX: J610.3 (P3)
- new net GPIO17/UART2_TX: J610.2 (P2)
- new net GPIO3/UART0_RX: J609.3 (P3)
- new net GPIO5/LED: J607.2 (P2)
Changed lines of the file:
@@
 EESchema Schematic File Version 2
-LIBS:HAP-IO-Card-rescue
 LIBS:power
 LIBS:device
@@
 Text GLabel 1800 1650 0    60   Input ~ 0
 VSPI_CS1
-Wire Wire Line
-	1800 1050 2200 1050
-Wire Wire Line
-	1800 1200 1900 1200
-Wire Wire Line
-	1900 1200 1900 1150
-Wire Wire Line
-	1900 1150 2300 1150
-Wire Wire Line
-	1800 1350 1900 1350
-Wire Wire Line
-	1900 1350 1900 1250
-Wire Wire Line
-	1900 1250 2400 1250
-Wire Wire Line
-	1800 1500 1950 1500
-Wire Wire Line
-	1950 1500 1950 1350
-Wire Wire Line
-	1950 1350 2500 1350
-$Comp
-L CONN_01X04 J24
+$Comp
+L CONN_01X04 J601
 U 1 1 5924A437
 P 2350 800
-F 0 "J24" V 2315 562 50  0000 R CNN
+F 0 "J601" V 2315 562 50  0000 R CNN
 F 1 "ISP0" V 2224 562 50  0000 R CNN
 F 2 "Pin_Headers:Pin_Header_Straight_1x04_Pitch2.54mm" H 2350 800 50  0001 C CNN
@@
 $EndComp
 $Comp
-L CONN_01X04 J25
+L CONN_01X04 J602
 U 1 1 5924A47C
 P 2350 1750
-F 0 "J25" V 2222 1512 50  0000 R CNN
+F 0 "J602" V 2222 1512 50  0000 R CNN
 F 1 "ISP1" V 2313 1512 50  0000 R CNN
 F 2 "Pin_Headers:Pin_Header_Straight_1x04_Pitch2.54mm" H 2350 1750 50  0001 C CNN
@@
 	0    -1   1    0
 $EndComp
-Wire Wire Line
-	2300 1000 2300 1550
-Wire Wire Line
-	2400 1000 2400 1550
-Wire Wire Line
-	2500 1350 2500 1000
-Connection ~ 2200 1050
-Wire Wire Line
-	2200 1000 2200 1550
-Connection ~ 2300 1150
-Connection ~ 2400 1250
-Wire Wire Line
-	1800 1650 2050 1650
-Wire Wire Line
-	2050 1650 2050 1500
-Wire Wire Line
-	2050 1500 2500 1500
-Wire Wire Line
-	2500 1500 2500 1550
-$Comp
-L CONN_01X01 J23
-U 1 1 5924AD72
-P 2000 2050
-F 0 "J23" H 2077 2091 50  0000 L CNN
-F 1 "Debug Log" H 2077 2000 50  0000 L CNN
-F 2 "" H 2000 2050 50  0001 C CNN
-F 3 "" H 2000 2050 50  0001 C CNN
-	1    2000 2050
-	1    0    0    -1
-$EndComp
-Text GLabel 1800 2050 0    60   Input ~ 0
-DebugLog
 Text GLabel 3750 1500 0    60   Input ~ 0
 JTAG:MTDI
@@
 ~RESET
 $Comp
-L AVR-JTAG-10 CON1
+L AVR-JTAG-10 CON601
 U 1 1 5924B014
 P 4450 1300
-F 0 "CON1" H 4424 1755 50  0000 C CNN
+F 0 "CON601" H 4424 1755 50  0000 C CNN
 F 1 "AVR-JTAG-10" H 4424 1664 50  0000 C CNN
 F 2 "Connectors:IDC_Header_Straight_10pins" V 3880 1320 50  0001 C CNN
@@
 $EndComp
 NoConn ~ 4250 1400
-Wire Wire Line
-	4500 1300 5200 1300
-Wire Wire Line
-	3900 1100 4250 1100
-Wire Wire Line
-	4500 1500 4900 1500
-Wire Wire Line
-	4850 1100 4500 1100
-Wire Wire Line
-	3750 1500 4250 1500
-Wire Wire Line
-	3750 1300 4250 1300
-Wire Wire Line
-	3800 1200 4250 1200
-Wire Wire Line
-	4850 1200 4500 1200
-Wire Wire Line
-	3900 1100 3900 1000
-Wire Wire Line
-	3900 1000 3750 1000
-Wire Wire Line
-	3800 1150 3750 1150
-Wire Wire Line
-	3800 1200 3800 1150
 NoConn ~ 4500 1400
 $Comp
@@
 	0    1    1    0
 $EndComp
-Text GLabel 3600 2100 0    60   Input ~ 0
-NeoPixel
-$Comp
-L CONN_01X01 J26
-U 1 1 5924B799
-P 3800 2100
-F 0 "J26" H 3877 2141 50  0000 L CNN
-F 1 "NeoPixel" H 3877 2050 50  0000 L CNN
-F 2 "" H 3800 2100 50  0001 C CNN
-F 3 "" H 3800 2100 50  0001 C CNN
-	1    3800 2100
-	1    0    0    -1
+Text GLabel 4150 2600 1    60   Input ~ 0
+GPIO5/LED
+Text GLabel 4800 2600 1    60   Input ~ 0
+GPIO0/Button
+Text GLabel 3550 2600 1    60   Input ~ 0
+GPI39
+Text GLabel 2950 2600 1    60   Input ~ 0
+GPI38
+$Comp
+L CONN_01X02 J603
+U 1 1 59270008
+P 3000 3150
+F 0 "J603" V 3100 3050 50  0000 L CNN
+F 1 "CONN_01X02" V 3200 2950 50  0000 L CNN
+F 2 "Pin_Headers:Pin_Header_Straight_1x02_Pitch2.54mm" H 3000 3150 50  0001 C CNN
+F 3 "" H 3000 3150 50  0001 C CNN
+	1    3000 3150
+	0    1    1    0
+$EndComp
+Text GLabel 5900 2800 1    60   Input ~ 0
+GPIO16/UART2_RX
+Text GLabel 6050 2800 1    60   Input ~ 0
+GPIO17/UART2_TX
+Text GLabel 5450 2800 1    60   Input ~ 0
+GPIO/1UART0_TX
+Text GLabel 5300 2800 1    60   Input ~ 0
+GPIO3/UART0_RX
+$Comp
+L GND #PWR083
+U 1 1 59270647
+P 3050 2950
+F 0 "#PWR083" H 3050 2700 50  0001 C CNN
+F 1 "GND" V 3055 2822 50  0000 R CNN
+F 2 "" H 3050 2950 50  0001 C CNN
+F 3 "" H 3050 2950 50  0001 C CNN
+	1    3050 2950
+	-1   0    0    1
+$EndComp
+$Comp
+L CONN_01X02 J604
+U 1 1 592706A6
+P 3600 3150
+F 0 "J604" V 3700 3050 50  0000 L CNN
+F 1 "CONN_01X02" V 3800 2950 50  0000 L CNN
+F 2 "Pin_Headers:Pin_Header_Straight_1x02_Pitch2.54mm" H 3600 3150 50  0001 C CNN
+F 3 "" H 3600 3150 50  0001 C CNN
+	1    3600 3150
+	0    1    1    0
+$EndComp
+Wire Wire Line
+	1800 1050 2200 1050
+Wire Wire Line
+	1800 1200 1900 1200
+Wire Wire Line
+	1900 1200 1900 1150
+Wire Wire Line
+	1900 1150 2300 1150
+Wire Wire Line
+	1800 1350 1900 1350
+Wire Wire Line
+	1900 1350 1900 1250
+Wire Wire Line
+	1900 1250 2400 1250
+Wire Wire Line
+	1800 1500 1950 1500
+Wire Wire Line
+	1950 1500 1950 1350
+Wire Wire Line
+	1950 1350 2500 1350
+Wire Wire Line
+	2300 1000 2300 1550
+Wire Wire Line
+	2400 1000 2400 1550
+Wire Wire Line
+	2500 1350 2500 1000
+Connection ~ 2200 1050
+Wire Wire Line
+	2200 1000 2200 1550
+Connection ~ 2300 1150
+Connection ~ 2400 1250
+Wire Wire Line
+	1800 1650 2050 1650
+Wire Wire Line
+	2050 1650 2050 1500
+Wire Wire Line
+	2050 1500 2500 1500
+Wire Wire Line
+	2500 1500 2500 1550
+Wire Wire Line
+	4500 1300 5200 1300
+Wire Wire Line
+	3900 1100 4250 1100
+Wire Wire Line
+	4500 1500 4900 1500
+Wire Wire Line
+	4850 1100 4500 1100
+Wire Wire Line
+	3750 1500 4250 1500
+Wire Wire Line
+	3750 1300 4250 1300
+Wire Wire Line
+	3800 1200 4250 1200
+Wire Wire Line
+	4850 1200 4500 1200
+Wire Wire Line
+	3900 1100 3900 1000
+Wire Wire Line
+	3900 1000 3750 1000
+Wire Wire Line
+	3800 1150 3750 1150
+Wire Wire Line
+	3800 1200 3800 1150
+Wire Wire Line
+	2950 2950 2950 2600
+Wire Wire Line
+	3550 2600 3550 2950
+$Comp
+L GND #PWR084
+U 1 1 59270781
+P 3650 2950
+F 0 "#PWR084" H 3650 2700 50  0001 C CNN
+F 1 "GND" V 3655 2822 50  0000 R CNN
+F 2 "" H 3650 2950 50  0001 C CNN
+F 3 "" H 3650 2950 50  0001 C CNN
+	1    3650 2950
+	-1   0    0    1
+$EndComp
+$Comp
+L CONN_01X02 J607
+U 1 1 592708FE
+P 4200 3150
+F 0 "J607" V 4300 3050 50  0000 L CNN
+F 1 "CONN_01X02" V 4400 2950 50  0000 L CNN
+F 2 "Pin_Headers:Pin_Header_Straight_1x02_Pitch2.54mm" H 4200 3150 50  0001 C CNN
+F 3 "" H 4200 3150 50  0001 C CNN
+	1    4200 3150
+	0    1    1    0
+$EndComp
+Wire Wire Line
+	4150 2600 4150 2950
+$Comp
+L GND #PWR085
+U 1 1 59270905
+P 4250 2950
+F 0 "#PWR085" H 4250 2700 50  0001 C CNN
+F 1 "GND" V 4255 2822 50  0000 R CNN
+F 2 "" H 4250 2950 50  0001 C CNN
+F 3 "" H 4250 2950 50  0001 C CNN
+	1    4250 2950
+	-1   0    0    1
+$EndComp
+$Comp
+L CONN_01X02 J608
+U 1 1 5927092F
+P 4850 3150
+F 0 "J608" V 4950 3050 50  0000 L CNN
+F 1 "CONN_01X02" V 5050 2950 50  0000 L CNN
+F 2 "Pin_Headers:Pin_Header_Straight_1x02_Pitch2.54mm" H 4850 3150 50  0001 C CNN
+F 3 "" H 4850 3150 50  0001 C CNN
+	1    4850 3150
+	0    1    1    0
+$EndComp
+Wire Wire Line
+	4800 2600 4800 2950
+$Comp
+L GND #PWR086
+U 1 1 59270936
+P 4900 2950
+F 0 "#PWR086" H 4900 2700 50  0001 C CNN
+F 1 "GND" V 4905 2822 50  0000 R CNN
+F 2 "" H 4900 2950 50  0001 C CNN
+F 3 "" H 4900 2950 50  0001 C CNN
+	1    4900 2950
+	-1   0    0    1
+$EndComp
+$Comp
+L CONN_01X03 J610
+U 1 1 59271357
+P 6050 3150
+F 0 "J610" V 6150 3050 50  0000 L CNN
+F 1 "CONN_01X03" V 6250 2950 50  0000 L CNN
+F 2 "Pin_Headers:Pin_Header_Straight_1x03_Pitch2.54mm" H 6050 3150 50  0001 C CNN
+F 3 "" H 6050 3150 50  0001 C CNN
+	1    6050 3150
+	0    1    1    0
+$EndComp
+$Comp
+L CONN_01X03 J609
+U 1 1 59271444
+P 5450 3150
+F 0 "J609" V 5550 3050 50  0000 L CNN
+F 1 "CONN_01X03" V 5650 2950 50  0000 L CNN
+F 2 "Pin_Headers:Pin_Header_Straight_1x03_Pitch2.54mm" H 5450 3150 50  0001 C CNN
+F 3 "" H 5450 3150 50  0001 C CNN
+	1    5450 3150
+	0    1    1    0
+$EndComp
+$Comp
+L GND #PWR087
+U 1 1 59271A0B
+P 5550 2950
+F 0 "#PWR087" H 5550 2700 50  0001 C CNN
+F 1 "GND" V 5555 2822 50  0000 R CNN
+F 2 "" H 5550 2950 50  0001 C CNN
+F 3 "" H 5550 2950 50  0001 C CNN
+	1    5550 2950
+	-1   0    0    1
+$EndComp
+Wire Wire Line
+	5450 2950 5450 2800
+Wire Wire Line
+	5350 2950 5350 2900
+Wire Wire Line
+	5350 2900 5300 2900
+Wire Wire Line
+	5300 2900 5300 2800
+Wire Wire Line
+	6050 2800 6050 2950
+Wire Wire Line
+	5950 2950 5950 2900
+Wire Wire Line
+	5950 2900 5900 2900
+Wire Wire Line
+	5900 2900 5900 2800
+$Comp
+L GND #PWR088
+U 1 1 59271B4E
+P 6150 2950
+F 0 "#PWR088" H 6150 2700 50  0001 C CNN
+F 1 "GND" V 6155 2822 50  0000 R CNN
+F 2 "" H 6150 2950 50  0001 C CNN
+F 3 "" H 6150 2950 50  0001 C CNN
+	1    6150 2950
+	-1   0    0    1
 $EndComp
 $EndSCHEMATC

Commit message: More layout
Parts:
- renumbered J607 to J605, J608 to J606, J609 to J607, J610 to J608
Changed lines of the file:
@@
 $EndComp
 $Comp
-L GND #PWR080
+L GND #PWR606
 U 1 1 5924B01B
 P 4900 1500
-F 0 "#PWR080" H 4900 1250 50  0001 C CNN
+F 0 "#PWR606" H 4900 1250 50  0001 C CNN
 F 1 "GND" V 4905 1372 50  0000 R CNN
 F 2 "" H 4900 1500 50  0001 C CNN
@@
 NoConn ~ 4500 1400
 $Comp
-L GND #PWR081
+L GND #PWR604
 U 1 1 5924B02F
 P 4850 1100
-F 0 "#PWR081" H 4850 850 50  0001 C CNN
+F 0 "#PWR604" H 4850 850 50  0001 C CNN
 F 1 "GND" V 4855 972 50  0000 R CNN
 F 2 "" H 4850 1100 50  0001 C CNN
@@
 $EndComp
 $Comp
-L +3V3 #PWR082
+L +3V3 #PWR605
 U 1 1 5924B035
 P 4850 1200
-F 0 "#PWR082" H 4850 1050 50  0001 C CNN
+F 0 "#PWR605" H 4850 1050 50  0001 C CNN
 F 1 "+3V3" V 4865 1328 50  0000 L CNN
 F 2 "" H 4850 1200 50  0001 C CNN
@@
 GPIO3/UART0_RX
 $Comp
-L GND #PWR083
+L GND #PWR601
 U 1 1 59270647
 P 3050 2950
-F 0 "#PWR083" H 3050 2700 50  0001 C CNN
+F 0 "#PWR601" H 3050 2700 50  0001 C CNN
 F 1 "GND" V 3055 2822 50  0000 R CNN
 F 2 "" H 3050 2950 50  0001 C CNN
@@
 	3550 2600 3550 2950
 $Comp
-L GND #PWR084
+L GND #PWR602
 U 1 1 59270781
 P 3650 2950
-F 0 "#PWR084" H 3650 2700 50  0001 C CNN
+F 0 "#PWR602" H 3650 2700 50  0001 C CNN
 F 1 "GND" V 3655 2822 50  0000 R CNN
 F 2 "" H 3650 2950 50  0001 C CNN
@@
 $EndComp
 $Comp
-L CONN_01X02 J607
+L CONN_01X02 J605
 U 1 1 592708FE
 P 4200 3150
-F 0 "J607" V 4300 3050 50  0000 L CNN
+F 0 "J605" V 4300 3050 50  0000 L CNN
 F 1 "CONN_01X02" V 4400 2950 50  0000 L CNN
 F 2 "Pin_Headers:Pin_Header_Straight_1x02_Pitch2.54mm" H 4200 3150 50  0001 C CNN
@@
 	4150 2600 4150 2950
 $Comp
-L GND #PWR085
+L GND #PWR603
 U 1 1 59270905
 P 4250 2950
-F 0 "#PWR085" H 4250 2700 50  0001 C CNN
+F 0 "#PWR603" H 4250 2700 50  0001 C CNN
 F 1 "GND" V 4255 2822 50  0000 R CNN
 F 2 "" H 4250 2950 50  0001 C CNN
@@
 $EndComp
 $Comp
-L CONN_01X02 J608
+L CONN_01X02 J606
 U 1 1 5927092F
 P 4850 3150
-F 0 "J608" V 4950 3050 50  0000 L CNN
+F 0 "J606" V 4950 3050 50  0000 L CNN
 F 1 "CONN_01X02" V 5050 2950 50  0000 L CNN
 F 2 "Pin_Headers:Pin_Header_Straight_1x02_Pitch2.54mm" H 4850 3150 50  0001 C CNN
@@
 	4800 2600 4800 2950
 $Comp
-L GND #PWR086
+L GND #PWR607
 U 1 1 59270936
 P 4900 2950
-F 0 "#PWR086" H 4900 2700 50  0001 C CNN
+F 0 "#PWR607" H 4900 2700 50  0001 C CNN
 F 1 "GND" V 4905 2822 50  0000 R CNN
 F 2 "" H 4900 2950 50  0001 C CNN
@@
 $EndComp
 $Comp
-L CONN_01X03 J610
+L CONN_01X03 J608
 U 1 1 59271357
 P 6050 3150
-F 0 "J610" V 6150 3050 50  0000 L CNN
+F 0 "J608" V 6150 3050 50  0000 L CNN
 F 1 "CONN_01X03" V 6250 2950 50  0000 L CNN
 F 2 "Pin_Headers:Pin_Header_Straight_1x03_Pitch2.54mm" H 6050 3150 50  0001 C CNN
@@
 $EndComp
 $Comp
-L CONN_01X03 J609
+L CONN_01X03 J607
 U 1 1 59271444
 P 5450 3150
-F 0 "J609" V 5550 3050 50  0000 L CNN
+F 0 "J607" V 5550 3050 50  0000 L CNN
 F 1 "CONN_01X03" V 5650 2950 50  0000 L CNN
 F 2 "Pin_Headers:Pin_Header_Straight_1x03_Pitch2.54mm" H 5450 3150 50  0001 C CNN
@@
 $EndComp
 $Comp
-L GND #PWR087
+L GND #PWR608
 U 1 1 59271A0B
 P 5550 2950
-F 0 "#PWR087" H 5550 2700 50  0001 C CNN
+F 0 "#PWR608" H 5550 2700 50  0001 C CNN
 F 1 "GND" V 5555 2822 50  0000 R CNN
 F 2 "" H 5550 2950 50  0001 C CNN
@@
 	5900 2900 5900 2800
 $Comp
-L GND #PWR088
+L GND #PWR609
 U 1 1 59271B4E
 P 6150 2950
-F 0 "#PWR088" H 6150 2700 50  0001 C CNN
+F 0 "#PWR609" H 6150 2700 50  0001 C CNN
 F 1 "GND" V 6155 2822 50  0000 R CNN
 F 2 "" H 6150 2950 50  0001 C CNN

Commit message: More layout
Parts:
- CON601: footprint Connectors:IDC_Header_Straight_10pins -> Pin_Headers:Pin_Header_Straight_2x06_Pitch2.54mm
Changed lines of the file:
@@
 F 0 "CON601" H 4424 1755 50  0000 C CNN
 F 1 "AVR-JTAG-10" H 4424 1664 50  0000 C CNN
-F 2 "Connectors:IDC_Header_Straight_10pins" V 3880 1320 50  0001 C CNN
+F 2 "Pin_Headers:Pin_Header_Straight_2x06_Pitch2.54mm" V 3880 1320 50  0001 C CNN
 F 3 "" H 4450 1300 50  0001 C CNN
 	1    4450 1300
@@
 $EndComp
 $Comp
-L GND #PWR606
+L GND #PWR095
 U 1 1 5924B01B
 P 4900 1500
-F 0 "#PWR606" H 4900 1250 50  0001 C CNN
+F 0 "#PWR095" H 4900 1250 50  0001 C CNN
 F 1 "GND" V 4905 1372 50  0000 R CNN
 F 2 "" H 4900 1500 50  0001 C CNN
@@
 NoConn ~ 4500 1400
 $Comp
-L GND #PWR604
+L GND #PWR096
 U 1 1 5924B02F
 P 4850 1100
-F 0 "#PWR604" H 4850 850 50  0001 C CNN
+F 0 "#PWR096" H 4850 850 50  0001 C CNN
 F 1 "GND" V 4855 972 50  0000 R CNN
 F 2 "" H 4850 1100 50  0001 C CNN
@@
 $EndComp
 $Comp
-L +3V3 #PWR605
+L +3V3 #PWR097
 U 1 1 5924B035
 P 4850 1200
-F 0 "#PWR605" H 4850 1050 50  0001 C CNN
+F 0 "#PWR097" H 4850 1050 50  0001 C CNN
 F 1 "+3V3" V 4865 1328 50  0000 L CNN
 F 2 "" H 4850 1200 50  0001 C CNN
@@
 GPIO3/UART0_RX
 $Comp
-L GND #PWR601
+L GND #PWR098
 U 1 1 59270647
 P 3050 2950
-F 0 "#PWR601" H 3050 2700 50  0001 C CNN
+F 0 "#PWR098" H 3050 2700 50  0001 C CNN
 F 1 "GND" V 3055 2822 50  0000 R CNN
 F 2 "" H 3050 2950 50  0001 C CNN
@@
 	3550 2600 3550 2950
 $Comp
-L GND #PWR602
+L GND #PWR099
 U 1 1 59270781
 P 3650 2950
-F 0 "#PWR602" H 3650 2700 50  0001 C CNN
+F 0 "#PWR099" H 3650 2700 50  0001 C CNN
 F 1 "GND" V 3655 2822 50  0000 R CNN
 F 2 "" H 3650 2950 50  0001 C CNN
@@
 	4150 2600 4150 2950
 $Comp
-L GND #PWR603
+L GND #PWR0100
 U 1 1 59270905
 P 4250 2950
-F 0 "#PWR603" H 4250 2700 50  0001 C CNN
+F 0 "#PWR0100" H 4250 2700 50  0001 C CNN
 F 1 "GND" V 4255 2822 50  0000 R CNN
 F 2 "" H 4250 2950 50  0001 C CNN
@@
 	4800 2600 4800 2950
 $Comp
-L GND #PWR607
+L GND #PWR0101
 U 1 1 59270936
 P 4900 2950
-F 0 "#PWR607" H 4900 2700 50  0001 C CNN
+F 0 "#PWR0101" H 4900 2700 50  0001 C CNN
 F 1 "GND" V 4905 2822 50  0000 R CNN
 F 2 "" H 4900 2950 50  0001 C CNN
@@
 $EndComp
 $Comp
-L GND #PWR608
+L GND #PWR0102
 U 1 1 59271A0B
 P 5550 2950
-F 0 "#PWR608" H 5550 2700 50  0001 C CNN
+F 0 "#PWR0102" H 5550 2700 50  0001 C CNN
 F 1 "GND" V 5555 2822 50  0000 R CNN
 F 2 "" H 5550 2950 50  0001 C CNN
@@
 	5900 2900 5900 2800
 $Comp
-L GND #PWR609
+L GND #PWR0103
 U 1 1 59271B4E
 P 6150 2950
-F 0 "#PWR609" H 6150 2700 50  0001 C CNN
+F 0 "#PWR0103" H 6150 2700 50  0001 C CNN
 F 1 "GND" V 6155 2822 50  0000 R CNN
 F 2 "" H 6150 2950 50  0001 C CNN
