File: KiCad/DigitalIO.sch (KiCad schematic (older format))
At the start: 105 parts, among them J1 DI1, J10 DO3/4, J11 DO5/6, J12 DO7/8, J2 DI2, J3 DI3, J4 DI4, J5 DI5, J6 DI6, J7 DI7, J8 DI8, J9 DO1/2, Q1 ZXTN25050DFHTA, Q2 ZXTN25050DFHTA, Q3 ZXTN25050DFHTA, Q4 ZXTN25050DFHTA, Q5 ZXTN25050DFHTA, Q6 ZXTN25050DFHTA, Q7 ZXTN25050DFHTA, Q8 ZXTN25050DFHTA, U1 LTV-354T, U2 LTV-354T, U3 LTV-354T, U4 LTV-354T, U5 LTV-354T, U6 LTV-354T, U7 LTV-354T, U8 LTV-354T, U9 MCP23017

Commit message: More work
Parts:
- D215: renamed from D15; footprint Diodes_THT:D_DO-15_P2.54mm_Vertical_KathodeUp -> Diodes_THT:D_DO-41_SOD81_P5.08mm_Vertical_KathodeUp
- D216: renamed from D16; footprint Diodes_THT:D_DO-15_P2.54mm_Vertical_KathodeUp -> Diodes_THT:D_DO-41_SOD81_P5.08mm_Vertical_KathodeUp
- D217: renamed from D17; footprint Diodes_THT:D_DO-15_P2.54mm_Vertical_KathodeUp -> Diodes_THT:D_DO-41_SOD81_P5.08mm_Vertical_KathodeUp
- D218: renamed from D18; footprint Diodes_THT:D_DO-15_P2.54mm_Vertical_KathodeUp -> Diodes_THT:D_DO-41_SOD81_P5.08mm_Vertical_KathodeUp
- D219: renamed from D19; footprint Diodes_THT:D_DO-15_P2.54mm_Vertical_KathodeUp -> Diodes_THT:D_DO-41_SOD81_P5.08mm_Vertical_KathodeUp
- D220: renamed from D20; footprint Diodes_THT:D_DO-15_P2.54mm_Vertical_KathodeUp -> Diodes_THT:D_DO-41_SOD81_P5.08mm_Vertical_KathodeUp
- D223: renamed from D23; footprint Diodes_THT:D_DO-15_P2.54mm_Vertical_KathodeUp -> Diodes_THT:D_DO-41_SOD81_P5.08mm_Vertical_KathodeUp
- D224: renamed from D24; footprint Diodes_THT:D_DO-15_P2.54mm_Vertical_KathodeUp -> Diodes_THT:D_DO-41_SOD81_P5.08mm_Vertical_KathodeUp
- renumbered C1 to C201, C2 to C202, C3 to C203, C4 to C204, C5 to C205, C6 to C206, C7 to C207, C8 to C208, C9 to C209, D8 to D201, D7 to D202, D6 to D203, D5 to D204, D4 to D205, D3 to D206, D2 to D207, D1 to D208, D9 to D209, D10 to D210, D11 to D211, D12 to D212, D13 to D213, D14 to D214, D21 to D221, D22 to D222, J1 to J201, J2 to J202, J3 to J203, J4 to J204, J5 to J205, J6 to J206, J7 to J207, J8 to J208, J9 to J209, J10 to J210, J11 to J211, J12 to J212, Q1 to Q201, Q2 to Q202, Q3 to Q203, Q4 to Q204, Q5 to Q205, Q6 to Q206, Q7 to Q207, Q8 to Q208, R1 to R201, R2 to R202, R3 to R203, R4 to R204, R5 to R205, R6 to R206, R7 to R207, R8 to R208, R16 to R209, R15 to R210, R14 to R211, R13 to R212, R12 to R213, R11 to R214, R10 to R215, R9 to R216, R17 to R217, R18 to R218, R19 to R219, R20 to R220, R21 to R221, R22 to R222, R23 to R223, R24 to R224, R25 to R225, R26 to R226, R27 to R227, R28 to R228, R29 to R229, R30 to R230, R31 to R231, R32 to R232, R33 to R233, R34 to R234, R35 to R235, R36 to R236, R37 to R237, R38 to R238, R39 to R239, R40 to R240, R41 to R241, R42 to R242, RN1 to RN201, U1 to U201, U2 to U202, U3 to U203, U4 to U204, U5 to U205, U6 to U206, U7 to U207, U8 to U208, U9 to U209
Other:
- moved on the sheet: D201, D202, D203, D204, D205, D206, D207, D208, R209, R210, R211, R212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

Commit message: More layout
Parts:
- removed RN201: 10k, Resistors_THT:R_Array_SIP9, symbol R_Network08
- added J213, J214, J215, J216: GND, Connectors_Terminal_Blocks:TerminalBlock_Pheonix_MPT-2.54mm_2pol, symbol Screw_Terminal_1x02
- added R243, R244, R245, R246, R247, R248, R249, R250: 10k, Resistors_SMD:R_0805, symbol R
Connections:
- net +3V3: now also R243.1, R244.1, R245.1, R246.1, R247.1, R248.1, R249.1, R250.1
- net DI1: now also R243.2
- net DI2: now also R244.2
- net DI3: now also R245.2
- net DI4: now also R246.2
- net DI5: now also R247.2
- net DI6: now also R248.2
- net DI7: now also R249.2
- net DI8: now also R250.2
- net GND: now also J209.2, J210.2, J211.2, J212.2, J213.2, J214.2, J215.2, J216.2
- net at D210.1 (K), D216.1 (K), Q202.3 (C): now also J210.1; no longer J209.2
- net at D211.1 (K), D217.1 (K), Q203.3 (C): now also J211.1; no longer J210.1
- net at D212.1 (K), D218.1 (K), Q204.3 (C): now also J212.1; no longer J210.2
- net at D213.1 (K), D219.1 (K), Q205.3 (C): now also J213.1; no longer J211.1
- net at D214.1 (K), D220.1 (K), Q206.3 (C): now also J214.1; no longer J211.2
- net at D221.1 (K), D223.1 (K), Q207.3 (C): now also J215.1; no longer J212.1
- net at D222.1 (K), D224.1 (K), Q208.3 (C): now also J216.1; no longer J212.2
Other:
- moved on the sheet: J210, J211, J212

Commit message: More layout
Connections:
- net GND: now also J209.1, J210.1, J211.1, J212.1, J213.1, J214.1, J215.1, J216.1; no longer J209.2, J210.2, J211.2, J212.2, J213.2, J214.2, J215.2, J216.2
- net at D209.1 (K), D215.1 (K), Q201.3 (C): now also J209.2; no longer J209.1
- net at D210.1 (K), D216.1 (K), Q202.3 (C): now also J210.2; no longer J210.1
- net at D211.1 (K), D217.1 (K), Q203.3 (C): now also J211.2; no longer J211.1
- net at D212.1 (K), D218.1 (K), Q204.3 (C): now also J212.2; no longer J212.1
- net at D213.1 (K), D219.1 (K), Q205.3 (C): now also J213.2; no longer J213.1
- net at D214.1 (K), D220.1 (K), Q206.3 (C): now also J214.2; no longer J214.1
- net at D221.1 (K), D223.1 (K), Q207.3 (C): now also J215.2; no longer J215.1
- net at D222.1 (K), D224.1 (K), Q208.3 (C): now also J216.2; no longer J216.1
Other:
- moved on the sheet: J209, J210, J211, J212, J213, J214, J215, J216
Changed lines of the file:
@@
 L Screw_Terminal_1x02 J209
 U 1 1 5923CE4C
-P 7350 1000
-F 0 "J209" H 7350 1250 50  0000 C TNN
-F 1 "DO1/2" V 7200 1000 50  0000 C TNN
-F 2 "Connectors_Terminal_Blocks:TerminalBlock_Pheonix_MPT-2.54mm_2pol" H 7350 775 50  0001 C CNN
-F 3 "" H 7325 1000 50  0001 C CNN
-	1    7350 1000
+P 7350 800
+F 0 "J209" H 7350 1050 50  0000 C TNN
+F 1 "DO1/2" V 7200 800 50  0000 C TNN
+F 2 "Connectors_Terminal_Blocks:TerminalBlock_Pheonix_MPT-2.54mm_2pol" H 7350 575 50  0001 C CNN
+F 3 "" H 7325 800 50  0001 C CNN
+	1    7350 800
 	-1   0    0    -1
 $EndComp
@@
 L Screw_Terminal_1x02 J210
 U 1 1 5924E202
-P 7350 2000
-F 0 "J210" H 7350 2250 50  0000 C TNN
-F 1 "DO3/4" V 7200 2000 50  0000 C TNN
-F 2 "Connectors_Terminal_Blocks:TerminalBlock_Pheonix_MPT-2.54mm_2pol" H 7350 1775 50  0001 C CNN
-F 3 "" H 7325 2000 50  0001 C CNN
-	1    7350 2000
+P 7350 1800
+F 0 "J210" H 7350 2050 50  0000 C TNN
+F 1 "DO3/4" V 7200 1800 50  0000 C TNN
+F 2 "Connectors_Terminal_Blocks:TerminalBlock_Pheonix_MPT-2.54mm_2pol" H 7350 1575 50  0001 C CNN
+F 3 "" H 7325 1800 50  0001 C CNN
+	1    7350 1800
 	-1   0    0    -1
 $EndComp
@@
 L Screw_Terminal_1x02 J211
 U 1 1 592504DE
-P 7350 3000
-F 0 "J211" H 7350 3250 50  0000 C TNN
-F 1 "DO5/6" V 7200 3000 50  0000 C TNN
-F 2 "Connectors_Terminal_Blocks:TerminalBlock_Pheonix_MPT-2.54mm_2pol" H 7350 2775 50  0001 C CNN
-F 3 "" H 7325 3000 50  0001 C CNN
-	1    7350 3000
+P 7350 2800
+F 0 "J211" H 7350 3050 50  0000 C TNN
+F 1 "DO5/6" V 7200 2800 50  0000 C TNN
+F 2 "Connectors_Terminal_Blocks:TerminalBlock_Pheonix_MPT-2.54mm_2pol" H 7350 2575 50  0001 C CNN
+F 3 "" H 7325 2800 50  0001 C CNN
+	1    7350 2800
 	-1   0    0    -1
 $EndComp
@@
 L Screw_Terminal_1x02 J212
 U 1 1 59251FF7
-P 7350 4000
-F 0 "J212" H 7350 4250 50  0000 C TNN
-F 1 "DO7/8" V 7200 4000 50  0000 C TNN
-F 2 "Connectors_Terminal_Blocks:TerminalBlock_Pheonix_MPT-2.54mm_2pol" H 7350 3775 50  0001 C CNN
-F 3 "" H 7325 4000 50  0001 C CNN
-	1    7350 4000
+P 7350 3800
+F 0 "J212" H 7350 4050 50  0000 C TNN
+F 1 "DO7/8" V 7200 3800 50  0000 C TNN
+F 2 "Connectors_Terminal_Blocks:TerminalBlock_Pheonix_MPT-2.54mm_2pol" H 7350 3575 50  0001 C CNN
+F 3 "" H 7325 3800 50  0001 C CNN
+	1    7350 3800
 	-1   0    0    -1
 $EndComp
@@
 L Screw_Terminal_1x02 J213
 U 1 1 592A5122
-P 7400 5000
-F 0 "J213" H 7400 5250 50  0000 C TNN
-F 1 "GND" V 7250 5000 50  0000 C TNN
-F 2 "Connectors_Terminal_Blocks:TerminalBlock_Pheonix_MPT-2.54mm_2pol" H 7400 4775 50  0001 C CNN
-F 3 "" H 7375 5000 50  0001 C CNN
-	1    7400 5000
+P 7400 4800
+F 0 "J213" H 7400 5050 50  0000 C TNN
+F 1 "GND" V 7250 4800 50  0000 C TNN
+F 2 "Connectors_Terminal_Blocks:TerminalBlock_Pheonix_MPT-2.54mm_2pol" H 7400 4575 50  0001 C CNN
+F 3 "" H 7375 4800 50  0001 C CNN
+	1    7400 4800
 	-1   0    0    -1
 $EndComp
@@
 L Screw_Terminal_1x02 J214
 U 1 1 592A5B41
-P 7400 6000
-F 0 "J214" H 7400 6250 50  0000 C TNN
-F 1 "GND" V 7250 6000 50  0000 C TNN
-F 2 "Connectors_Terminal_Blocks:TerminalBlock_Pheonix_MPT-2.54mm_2pol" H 7400 5775 50  0001 C CNN
-F 3 "" H 7375 6000 50  0001 C CNN
-	1    7400 6000
+P 7400 5800
+F 0 "J214" H 7400 6050 50  0000 C TNN
+F 1 "GND" V 7250 5800 50  0000 C TNN
+F 2 "Connectors_Terminal_Blocks:TerminalBlock_Pheonix_MPT-2.54mm_2pol" H 7400 5575 50  0001 C CNN
+F 3 "" H 7375 5800 50  0001 C CNN
+	1    7400 5800
 	-1   0    0    -1
 $EndComp
@@
 L Screw_Terminal_1x02 J215
 U 1 1 592A770A
-P 10500 1050
-F 0 "J215" H 10500 1300 50  0000 C TNN
-F 1 "GND" V 10350 1050 50  0000 C TNN
-F 2 "Connectors_Terminal_Blocks:TerminalBlock_Pheonix_MPT-2.54mm_2pol" H 10500 825 50  0001 C CNN
-F 3 "" H 10475 1050 50  0001 C CNN
-	1    10500 1050
+P 10500 850
+F 0 "J215" H 10500 1100 50  0000 C TNN
+F 1 "GND" V 10350 850 50  0000 C TNN
+F 2 "Connectors_Terminal_Blocks:TerminalBlock_Pheonix_MPT-2.54mm_2pol" H 10500 625 50  0001 C CNN
+F 3 "" H 10475 850 50  0001 C CNN
+	1    10500 850
 	-1   0    0    -1
 $EndComp
@@
 L Screw_Terminal_1x02 J216
 U 1 1 592A7710
-P 10450 2050
-F 0 "J216" H 10450 2300 50  0000 C TNN
-F 1 "GND" V 10300 2050 50  0000 C TNN
-F 2 "Connectors_Terminal_Blocks:TerminalBlock_Pheonix_MPT-2.54mm_2pol" H 10450 1825 50  0001 C CNN
-F 3 "" H 10425 2050 50  0001 C CNN
-	1    10450 2050
+P 10450 1850
+F 0 "J216" H 10450 2100 50  0000 C TNN
+F 1 "GND" V 10300 1850 50  0000 C TNN
+F 2 "Connectors_Terminal_Blocks:TerminalBlock_Pheonix_MPT-2.54mm_2pol" H 10450 1625 50  0001 C CNN
+F 3 "" H 10425 1850 50  0001 C CNN
+	1    10450 1850
 	-1   0    0    -1
 $EndComp
 $Comp
-L GND #PWR?
+L GND #PWR049
 U 1 1 592B1673
-P 7150 1100
-F 0 "#PWR?" H 7150 850 50  0001 C CNN
-F 1 "GND" H 7155 927 50  0000 C CNN
-F 2 "" H 7150 1100 50  0001 C CNN
-F 3 "" H 7150 1100 50  0001 C CNN
-	1    7150 1100
-	0    1    1    0
-$EndComp
-$Comp
-L GND #PWR?
+P 7150 700
+F 0 "#PWR049" H 7150 450 50  0001 C CNN
+F 1 "GND" H 7155 527 50  0000 C CNN
+F 2 "" H 7150 700 50  0001 C CNN
+F 3 "" H 7150 700 50  0001 C CNN
+	1    7150 700
+	0    1    1    0
+$EndComp
+$Comp
+L GND #PWR050
 U 1 1 592B18C2
-P 7150 2100
-F 0 "#PWR?" H 7150 1850 50  0001 C CNN
-F 1 "GND" H 7155 1927 50  0000 C CNN
-F 2 "" H 7150 2100 50  0001 C CNN
-F 3 "" H 7150 2100 50  0001 C CNN
-	1    7150 2100
-	0    1    1    0
-$EndComp
-$Comp
-L GND #PWR?
+P 7150 1700
+F 0 "#PWR050" H 7150 1450 50  0001 C CNN
+F 1 "GND" H 7155 1527 50  0000 C CNN
+F 2 "" H 7150 1700 50  0001 C CNN
+F 3 "" H 7150 1700 50  0001 C CNN
+	1    7150 1700
+	0    1    1    0
+$EndComp
+$Comp
+L GND #PWR051
 U 1 1 592B21DD
-P 7150 3100
-F 0 "#PWR?" H 7150 2850 50  0001 C CNN
-F 1 "GND" H 7155 2927 50  0000 C CNN
-F 2 "" H 7150 3100 50  0001 C CNN
-F 3 "" H 7150 3100 50  0001 C CNN
-	1    7150 3100
-	0    1    1    0
-$EndComp
-$Comp
-L GND #PWR?
+P 7150 2700
+F 0 "#PWR051" H 7150 2450 50  0001 C CNN
+F 1 "GND" H 7155 2527 50  0000 C CNN
+F 2 "" H 7150 2700 50  0001 C CNN
+F 3 "" H 7150 2700 50  0001 C CNN
+	1    7150 2700
+	0    1    1    0
+$EndComp
+$Comp
+L GND #PWR052
 U 1 1 592B2BE0
-P 7150 4100
-F 0 "#PWR?" H 7150 3850 50  0001 C CNN
-F 1 "GND" H 7155 3927 50  0000 C CNN
-F 2 "" H 7150 4100 50  0001 C CNN
-F 3 "" H 7150 4100 50  0001 C CNN
-	1    7150 4100
-	0    1    1    0
-$EndComp
-$Comp
-L GND #PWR?
+P 7150 3700
+F 0 "#PWR052" H 7150 3450 50  0001 C CNN
+F 1 "GND" H 7155 3527 50  0000 C CNN
+F 2 "" H 7150 3700 50  0001 C CNN
+F 3 "" H 7150 3700 50  0001 C CNN
+	1    7150 3700
+	0    1    1    0
+$EndComp
+$Comp
+L GND #PWR053
 U 1 1 592B3243
-P 7200 5100
-F 0 "#PWR?" H 7200 4850 50  0001 C CNN
-F 1 "GND" H 7205 4927 50  0000 C CNN
-F 2 "" H 7200 5100 50  0001 C CNN
-F 3 "" H 7200 5100 50  0001 C CNN
-	1    7200 5100
-	0    1    1    0
-$EndComp
-$Comp
-L GND #PWR?
+P 7200 4700
+F 0 "#PWR053" H 7200 4450 50  0001 C CNN
+F 1 "GND" H 7205 4527 50  0000 C CNN
+F 2 "" H 7200 4700 50  0001 C CNN
+F 3 "" H 7200 4700 50  0001 C CNN
+	1    7200 4700
+	0    1    1    0
+$EndComp
+$Comp
+L GND #PWR054
 U 1 1 592B3A02
-P 7200 6100
-F 0 "#PWR?" H 7200 5850 50  0001 C CNN
-F 1 "GND" H 7205 5927 50  0000 C CNN
-F 2 "" H 7200 6100 50  0001 C CNN
-F 3 "" H 7200 6100 50  0001 C CNN
-	1    7200 6100
-	0    1    1    0
-$EndComp
-$Comp
-L GND #PWR?
+P 7200 5700
+F 0 "#PWR054" H 7200 5450 50  0001 C CNN
+F 1 "GND" H 7205 5527 50  0000 C CNN
+F 2 "" H 7200 5700 50  0001 C CNN
+F 3 "" H 7200 5700 50  0001 C CNN
+	1    7200 5700
+	0    1    1    0
+$EndComp
+$Comp
+L GND #PWR055
 U 1 1 592B3AF5
-P 10250 2150
-F 0 "#PWR?" H 10250 1900 50  0001 C CNN
-F 1 "GND" H 10255 1977 50  0000 C CNN
-F 2 "" H 10250 2150 50  0001 C CNN
-F 3 "" H 10250 2150 50  0001 C CNN
-	1    10250 2150
-	0    1    1    0
-$EndComp
-$Comp
-L GND #PWR?
+P 10250 1750
+F 0 "#PWR055" H 10250 1500 50  0001 C CNN
+F 1 "GND" H 10255 1577 50  0000 C CNN
+F 2 "" H 10250 1750 50  0001 C CNN
+F 3 "" H 10250 1750 50  0001 C CNN
+	1    10250 1750
+	0    1    1    0
+$EndComp
+$Comp
+L GND #PWR056
 U 1 1 592B53EC
-P 10300 1150
-F 0 "#PWR?" H 10300 900 50  0001 C CNN
-F 1 "GND" H 10305 977 50  0000 C CNN
-F 2 "" H 10300 1150 50  0001 C CNN
-F 3 "" H 10300 1150 50  0001 C CNN
-	1    10300 1150
-	0    1    1    0
-$EndComp
+P 10300 750
+F 0 "#PWR056" H 10300 500 50  0001 C CNN
+F 1 "GND" H 10305 577 50  0000 C CNN
+F 2 "" H 10300 750 50  0001 C CNN
+F 3 "" H 10300 750 50  0001 C CNN
+	1    10300 750
+	0    1    1    0
+$EndComp
