File: KiCad/HAP-IO-Card.kicad_pcb (KiCad board)
At the start: 2 copper layers, 110 x 72 mm, 229 parts, among them CON601 AVR-JTAG-10, J201 TE_Connectivity_1-282834-0, J202 TE_Connectivity_282834-6, J203 GS3, J204 GS3, J205 GS3, J206 GS3, J207 GS3, J208 GS3, J209 GS3, J210 GS3, J211 TE_Connectivity_282834-6, J212 TE_Connectivity_1-282834-0, J401 TE_Connectivity_1-282834-0, J402 TE_Connectivity_282834-6, J501 TE_Connectivity_282834-3, J502 CONN_01X03_FEMALE, J601 ISP0, J602 ISP1, J603 CONN_01X02, J604 CONN_01X02, J605 CONN_01X02, J606 CONN_01X02, J607 CONN_01X03, J608 CONN_01X03, J701 5V_I/O_2, J702 5V_I/O_1, J703 NEO1, J704 NEO2, J705 NEO3, J706 NEO4, J707 CONN_01X03, Q201 ZXTN25050DFHTA, Q202 ZXTN25050DFHTA, Q203 ZXTN25050DFHTA, Q204 ZXTN25050DFHTA, Q205 ZXTN25050DFHTA, Q206 ZXTN25050DFHTA, Q207 ZXTN25050DFHTA, Q208 ZXTN25050DFHTA, U201 LTV-354T, U202 LTV-354T, U203 LTV-354T, U204 LTV-354T, U205 LTV-354T, U206 LTV-354T, U207 LTV-354T, U208 LTV-354T, U209 MCP23017, U401 ADS1115IDGST, U402 ADS1115IDGST, U501 LM1086-5V, U502 LM1086-3.3V, U701 TXB0102DCT

Commit message: Routing
Parts:
- moved C409 16.1 mm to (124.3, 55.7), turned to 270 degrees
- moved C410 14.1 mm to (113.4, 66.1), turned to 270 degrees
- moved U402 10.3 mm to (118.6, 55.9), turned to 180 degrees
- moved U401 10.2 mm to (118.6, 66.2), turned to 180 degrees
- moved R423 0.38 mm to (110.8, 49.7), turned to 90 degrees
- turned R409 to 90 degrees
Connections:
- net Net-(D501-Pad1) renamed /Powersupply/12V_PWR2
Routing:
- net POWER5V: track 0.00 -> 283.7 mm, vias 0 -> 2
- net POWER3V3: track 0.00 -> 73.6 mm, vias 0 -> 4
- net Sense8: track 0.00 -> 28.0 mm, vias 0 -> 1
- net Net-(C408-Pad2): track 0.00 -> 24.5 mm
- net +12V: track 0.00 -> 24.2 mm
- net Sense1: track 0.00 -> 21.3 mm, vias 0 -> 1
- net Net-(C401-Pad2): track 0.00 -> 21.1 mm
- net Net-(C407-Pad2): track 0.00 -> 20.2 mm
- net Net-(C402-Pad2): track 0.00 -> 19.4 mm
- net Net-(C703-Pad1): track 0.00 -> 19.2 mm
- net Net-(C404-Pad2): track 0.00 -> 19.1 mm
- net Net-(C403-Pad2): track 0.00 -> 19.0 mm
- net Net-(C406-Pad2): track 0.00 -> 18.6 mm
- net /Sense Inputs/Sense8_DUT: track 0.00 -> 18.5 mm
- net /Sense Inputs/Sense6_DUT: track 0.00 -> 18.5 mm
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